File: kicad/StackOverChonk.kicad_pcb (KiCad board)
At the start: 2 copper layers, 138.9 x 113.2 mm, 93 parts

Commit message: PCB Routed
Routing:
- net VCC: track 101.4 -> 782.8 mm, vias 27 -> 29
- net (no net): track 337.7 -> 0.00 mm
- net P1: track 33.1 -> 237.4 mm, vias 4 -> 5
- net P0: track 33.1 -> 219.9 mm, vias 4 -> 5
- net P5: track 41.3 -> 215.6 mm
- net P18: track 13.2 -> 187.2 mm, vias 6 -> 7
- net P4: track 33.1 -> 204.2 mm
- net P19: track 13.2 -> 172.5 mm, vias 6 -> 7
- net P15: track 6.60 -> 164.3 mm, vias 3 -> 4
- net P7: track 41.3 -> 188.5 mm
- net P20: track 13.2 -> 156.8 mm, vias 6 -> 7
- net P8: track 41.3 -> 179.3 mm
- net P21: track 13.2 -> 148.8 mm, vias 6 -> 7
- net P6: track 6.76 -> 112.7 mm, vias 1 -> 2
- net LED_3: track 13.5 -> 94.3 mm
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